File: ESP01M_Carrier.brd (EAGLE design)
At the start: 15.2 x 22.9 mm, 3 parts

Commit message: uipdate gerber & pcb layout
Connections:
- net N$1 renamed RST
- net N$10 renamed GND
- net N$11 renamed VDD
- net N$12 renamed TXD
- net N$13 renamed RXD
- net N$14 renamed IO13
- net N$15 renamed IO15
- net N$16 renamed IO2
- net N$17 renamed IO0
- net N$18 renamed EN
- net N$2 renamed IO16
- net N$3 renamed ADC
- net N$4 renamed IO14
- net N$5 renamed IO12
- net N$6 renamed IO5
- net N$7 renamed IO10
- net N$8 renamed IO9
- net N$9 renamed IO4
Other:
- board text added: "ADC"
- board text added: "EN"
- board text added: "GND"
- board text added: "IO0"
- board text added: "IO10"
- board text added: "IO12"
- board text added: "IO13"
- board text added: "IO14"
- board text added: "IO15"
- board text added: "IO16"
- board text added: "IO2"
- board text added: "IO4"
- board text added: "IO5"
- board text added: "IO9"
- board text added: "RST"
- board text added: "RXD"
- board text added: "TXD"
- board text added: "VDD"
Changed lines of the file:
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@@
 <?xml version="1.0" encoding="utf-8"?>
 <!DOCTYPE eagle SYSTEM "eagle.dtd">
-<eagle version="7.7.0">
+<eagle version="9.0.1">
 <drawing>
 <settings>
 <setting alwaysvectorfont="yes"/>
+<setting keepoldvectorfont="yes"/>
 <setting verticaltext="up"/>
 </settings>
-<grid distance="0.1" unitdist="mm" unit="mm" style="lines" multiple="1" display="yes" altdistance="0.025" altunitdist="inch" altunit="mm"/>
+<grid distance="0.1" unitdist="mm" unit="mm" style="lines" multiple="1" display="yes" altdistance="0.1" altunitdist="mm" altunit="mm"/>
 <layers>
 <layer number="1" name="Top" color="4" fill="1" visible="yes" active="yes"/>
@@
 <layer number="45" name="Holes" color="7" fill="1" visible="no" active="yes"/>
 <layer number="46" name="Milling" color="3" fill="1" visible="no" active="yes"/>
-<layer number="47" name="Measures" color="7" fill="1" visible="no" active="yes"/>
+<layer number="47" name="Measures" color="7" fill="1" visible="yes" active="yes"/>
 <layer number="48" name="Document" color="7" fill="1" visible="yes" active="yes"/>
 <layer number="49" name="Reference" color="7" fill="1" visible="yes" active="yes"/>
@@
 <wire x1="15.22" y1="22.938" x2="0" y2="22.938" width="0" layer="20"/>
 <wire x1="0" y1="22.938" x2="0" y2="0" width="0" layer="20"/>
+<text x="10.4" y="21.2" size="0.8128" layer="25" font="vector">GND</text>
+<text x="10.4" y="18.6" size="0.8128" layer="25" font="vector" distance="40">VDD</text>
+<text x="10.4" y="16.2" size="0.8128" layer="25" font="vector" distance="40">TXD</text>
+<text x="10.4" y="13.6" size="0.8128" layer="25" font="vector" distance="40">RXD</text>
+<text x="9.9" y="11" size="0.8128" layer="25" font="vector" distance="40">IO13</text>
+<text x="9.9" y="8.5" size="0.8128" layer="25" font="vector" distance="40">IO15</text>
+<text x="10.6" y="6" size="0.8128" layer="25" font="vector" distance="40">IO2</text>
+<text x="10.6" y="3.4" size="0.8128" layer="25" font="vector" distance="40">IO0</text>
+<text x="11.1" y="0.9" size="0.8128" layer="25" font="vector" distance="40">EN</text>
+<text x="2.8" y="21.2" size="0.8128" layer="25" font="vector">RST</text>
+<text x="2.8" y="18.6" size="0.8128" layer="25" font="vector">IO16</text>
+<text x="2.8" y="16.2" size="0.8128" layer="25" font="vector">ADC</text>
+<text x="2.8" y="13.6" size="0.8128" layer="25" font="vector">IO14</text>
+<text x="2.8" y="11" size="0.8128" layer="25" font="vector">IO12</text>
+<text x="2.8" y="8.5" size="0.8128" layer="25" font="vector">IO5</text>
+<text x="2.8" y="6" size="0.8128" layer="25" font="vector">IO10</text>
+<text x="2.8" y="3.4" size="0.8128" layer="25" font="vector">IO9</text>
+<text x="2.8" y="0.9" size="0.8128" layer="25" font="vector">IO4</text>
+<dimension x1="7.35" y1="13.5" x2="8.15" y2="13.4" x3="7.75" y3="25" textsize="1.778" layer="47" dtype="horizontal"/>
+<dimension x1="7.62" y1="4.08" x2="8.1" y2="19.1" x3="21.4" y3="11.59" textsize="1.778" layer="47" dtype="vertical"/>
 </plain>
 <attributes>
@@
 <param name="dpMaxLengthDifference" value="10mm"/>
 <param name="dpGapFactor" value="2.5"/>
-<param name="checkGrid" value="0"/>
 <param name="checkAngle" value="0"/>
 <param name="checkFont" value="1"/>
 <param name="checkRestrict" value="1"/>
+<param name="checkStop" value="0"/>
+<param name="checkValues" value="0"/>
 <param name="useDiameter" value="13"/>
 <param name="maxErrors" value="50"/>
@@
 </element>
 <element name="ESP-01M" library="Smart_Rak" package="ESP-01M" value="" x="7.62" y="4.08" smashed="yes">
-<attribute name="NAME" x="5.62" y="2.08" size="0.6096" layer="25"/>
+<attribute name="NAME" x="5.72" y="1.98" size="0.6096" layer="25"/>
 <attribute name="VALUE" x="5.52" y="20.08" size="1.016" layer="25"/>
 </element>
 </elements>
 <signals>
-<signal name="N$1">
+<signal name="RST">
 <contactref element="__" pad="9"/>
 <contactref element="ESP-01M" pad="18"/>
@@
 <wire x1="4.98" y1="17.88" x2="1.27" y2="21.59" width="0.3048" layer="16"/>
 </signal>
-<signal name="N$2">
+<signal name="IO16">
 <contactref element="__" pad="8"/>
 <contactref element="ESP-01M" pad="17"/>
@@
 <wire x1="4.04" y1="16.28" x2="1.27" y2="19.05" width="0.3048" layer="16"/>
 </signal>
-<signal name="N$3">
+<signal name="ADC">
 <contactref element="__" pad="7"/>
 <contactref element="ESP-01M" pad="16"/>
@@
 <wire x1="3.1" y1="14.68" x2="1.27" y2="16.51" width="0.3048" layer="16"/>
 </signal>
-<signal name="N$4">
+<signal name="IO14">
 <contactref element="__" pad="6"/>
 <contactref element="ESP-01M" pad="15"/>
@@
 <wire x1="2.16" y1="13.08" x2="1.27" y2="13.97" width="0.3048" layer="16"/>
 </signal>
-<signal name="N$5">
+<signal name="IO12">
 <contactref element="__" pad="5"/>
 <contactref element="ESP-01M" pad="14"/>
@@
 <wire x1="1.32" y1="11.48" x2="1.27" y2="11.43" width="0.3048" layer="16"/>
 </signal>
-<signal name="N$6">
+<signal name="IO5">
 <contactref element="__" pad="4"/>
 <contactref element="ESP-01M" pad="13"/>
@@
 <wire x1="2.26" y1="9.88" x2="1.27" y2="8.89" width="0.3048" layer="16"/>
 </signal>
-<signal name="N$7">
+<signal name="IO10">
 <contactref element="__" pad="3"/>
 <contactref element="ESP-01M" pad="12"/>
@@
 <wire x1="3.2" y1="8.28" x2="1.27" y2="6.35" width="0.3048" layer="16"/>
 </signal>
-<signal name="N$8">
+<signal name="IO9">
 <contactref element="__" pad="2"/>
 <contactref element="ESP-01M" pad="11"/>
@@
 <wire x1="4.14" y1="6.68" x2="1.27" y2="3.81" width="0.3048" layer="16"/>
 </signal>
-<signal name="N$9">
+<signal name="IO4">
 <contactref element="__" pad="1"/>
 <contactref element="ESP-01M" pad="10"/>
@@
 <wire x1="5.08" y1="5.08" x2="1.27" y2="1.27" width="0.3048" layer="16"/>
 </signal>
-<signal name="N$10">
+<signal name="GND">
 <contactref element="ESP-01M" pad="1"/>
 <contactref element="_" pad="1"/>
@@
 <wire x1="10.26" y1="17.88" x2="13.97" y2="21.59" width="0.3048" layer="16"/>
 </signal>
-<signal name="N$11">
+<signal name="VDD">
 <contactref element="ESP-01M" pad="2"/>
 <contactref element="_" pad="2"/>
@@
 <wire x1="11.2" y1="16.28" x2="13.97" y2="19.05" width="0.3048" layer="16"/>
 </signal>
-<signal name="N$12">
+<signal name="TXD">
 <contactref element="ESP-01M" pad="3"/>
 <contactref element="_" pad="3"/>
@@
 <wire x1="12.14" y1="14.68" x2="13.97" y2="16.51" width="0.3048" layer="16"/>
 </signal>
-<signal name="N$13">
+<signal name="RXD">
 <contactref element="ESP-01M" pad="4"/>
 <contactref element="_" pad="4"/>
@@
 <wire x1="13.08" y1="13.08" x2="13.97" y2="13.97" width="0.3048" layer="16"/>
 </signal>
-<signal name="N$14">
+<signal name="IO13">
 <contactref element="ESP-01M" pad="5"/>
 <contactref element="_" pad="5"/>
@@
 <wire x1="13.92" y1="11.48" x2="13.97" y2="11.43" width="0.3048" layer="16"/>
 </signal>
-<signal name="N$15">
+<signal name="IO15">
 <contactref element="ESP-01M" pad="6"/>
 <contactref element="_" pad="6"/>
@@
 <wire x1="12.98" y1="9.88" x2="13.97" y2="8.89" width="0.3048" layer="16"/>
 </signal>
-<signal name="N$16">
+<signal name="IO2">
 <contactref element="ESP-01M" pad="7"/>
 <contactref element="_" pad="7"/>
@@
 <wire x1="12.04" y1="8.28" x2="13.97" y2="6.35" width="0.3048" layer="16"/>
 </signal>
-<signal name="N$17">
+<signal name="IO0">
 <contactref element="ESP-01M" pad="8"/>
 <contactref element="_" pad="8"/>
@@
 <wire x1="11.1" y1="6.68" x2="13.97" y2="3.81" width="0.3048" layer="16"/>
 </signal>
-<signal name="N$18">
+<signal name="EN">
 <contactref element="ESP-01M" pad="9"/>
 <contactref element="_" pad="9"/>
